File: avs-mod-shield/hardware/avs-mod-shield.kicad_pcb (KiCad board)
At the start: 2 copper layers, 101.6 x 53.3 mm, 27 parts, among them P1 Digital, P10 CONN_1, P11 CONN_1, P12 CONN_1, P13 CONN_1, P2 Power, P3 Analog, P4 Analog, P5 PWM, P6 PWM, P7 Communication, P8 CONN_1, P9 CONN_1

Commit message: NOTICKET: Finalized Shield to Revision 0.1
- Finalized Schematic
- Finalized Layout
- Created Gerber Files
- Created pdf
Parts:
- added SP1: SPEAKER, Buzzers_Beepers:Buzzer_12x9.5RM7.6, F.Cu at (162.6, 80.0)
- added X1: CONN_01X02, Terminal_Blocks:TerminalBlock_WAGO-804_RM5mm_2pol, F.Cu at (108.1, 70.7)
- moved XR1 25.5 mm to (184.7, 73.9), turned to 0 degrees
- moved XV1 4.02 mm to (119.4, 78.7)
- moved XV2 4.02 mm to (125.7, 78.7)
- moved XV3 4.02 mm to (132.1, 78.7)
- moved XV4 4.02 mm to (138.4, 78.7)
- moved XV5 4.02 mm to (144.8, 78.7)
- moved XV6 4.02 mm to (151.1, 78.7)
Connections:
- P1 pad 11: /P0 -> /P7
- P1 pad 12: /P1 -> /P6
- P1 pad 13: /P2 -> /P5
- P1 pad 14: /P3 -> /P4
- P1 pad 15: /P4 -> /P3
- P1 pad 16: /P5 -> /P2
- P1 pad 17: /P6 -> /P1
- P1 pad 18: /P7 -> /P0
- P1 pad 19: (no net) -> LD1
- P1 pad 20: (no net) -> //G
- P1 pad 21: (no net) -> LD2
- P1 pad 23: (no net) -> /TA7
- P1 pad 24: (no net) -> /TA6
- P1 pad 25: (no net) -> /TA5
- P1 pad 26: (no net) -> /TA4
- P1 pad 27: (no net) -> /TA3
- P1 pad 28: (no net) -> /TA2
- P1 pad 29: (no net) -> /TA1
- P1 pad 30: (no net) -> /TA0
- P2 pad 2: (no net) -> +5V
- P5 pad 10: (no net) -> /TW6
- P5 pad 9: (no net) -> BUZZER
- P6 pad 1: (no net) -> /TW5
- P6 pad 2: (no net) -> /TW4
- P6 pad 3: (no net) -> /TW3
- P6 pad 4: (no net) -> /TW2
- P6 pad 5: (no net) -> /TW1
- P6 pad 6: (no net) -> /TW0
- XD1 pad 6: (no net) -> LD2
- XD1 pad 7: (no net) -> LD1
- XR1 pad 1: (no net) -> /TW0
- XR1 pad 10: (no net) -> /TW5
- XR1 pad 12: (no net) -> /TW6
- XR1 pad 13: (no net) -> /TA0
- XR1 pad 14: (no net) -> /TA1
- XR1 pad 15: (no net) -> /TA2
- XR1 pad 16: (no net) -> /TA3
- XR1 pad 17: (no net) -> /TA4
- XR1 pad 18: (no net) -> /TA5
- XR1 pad 19: (no net) -> /TA6
- XR1 pad 2: (no net) -> /TW1
- XR1 pad 20: (no net) -> /TA7
- XR1 pad 5: (no net) -> /TW2
- XR1 pad 6: (no net) -> /TW3
- XR1 pad 9: (no net) -> /TW4
Routing:
- net //G: track 61.6 -> 119.6 mm
- net /TW6: track 0.00 -> 52.7 mm
- net /TW5: track 0.00 -> 46.8 mm
- net /TW4: track 0.00 -> 39.6 mm
- net /TW3: track 0.00 -> 37.4 mm
- net /P5: track 94.5 -> 131.4 mm
- net /P0: track 87.8 -> 124.4 mm
- net /P1: track 93.5 -> 126.5 mm
- net LD1: track 0.00 -> 32.8 mm
- net /TW2: track 0.00 -> 31.3 mm
- net LD2: track 0.00 -> 31.3 mm
- net /TW1: track 0.00 -> 30.3 mm
- net /P2: track 87.1 -> 114.3 mm
- net /P6: track 90.2 -> 115.3 mm
- net /TA6: track 0.00 -> 24.5 mm
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Other:
- board text added: "+"
- board text added: "-"
- board text added: "- + -"
- board text added: "AVS 1280"
- board text added: "Arduino Mega Shield"
- board text added: "Rev. 0.1 2017 DC1MIL (andz) CC-BY-SA 4.0"
