File: avs-mod-shield/hardware/avs-mod-shield.sch (KiCad schematic (older format))
At the start: 27 parts, among them P1 Digital, P10 CONN_1, P11 CONN_1, P12 CONN_1, P13 CONN_1, P2 Power, P3 Analog, P4 Analog, P5 PWM, P6 PWM, P7 Communication, P8 CONN_1, P9 CONN_1

Commit message: NOTICKET: Finalized Shield to Revision 0.1
- Finalized Schematic
- Finalized Layout
- Created Gerber Files
- Created pdf
Parts:
- added SP1: SPEAKER, Buzzers_Beepers:Buzzer_12x9.5RM7.6, symbol SPEAKER
- added X1: CONN_01X02, Terminal_Blocks:TerminalBlock_WAGO-804_RM5mm_2pol, symbol CONN_01X02
Connections:
- net labels added: 9, BUZZER
- net labels removed: 2(**), 26, 27, 28, 29, 3(**), 30, 31, 32, 33, 34, 36, 37, 4(**), 5(**), 6(**), 7(**), 8(**), 9(**)
- wire segments 287 -> 288
Other:
- note added: "AVS 1280 Bus Connectors"
- note added: "Arduino Mega Rev 3"
- note added: "Display\nConnector"
- note added: "Keypad\nConnector"
- note added: "Power Connectors"
- note removed: "Shield for Arduino Mega Rev 3"
